File: terminal.sch (KiCad schematic (older format))
At the start: 37 parts, among them J1 VGA Connector, J2 Mini-DIN-6, J3 UART Connector, J4 DEBUG UART HEADER, J5 Power connector, Q1 BSS138, Q2 BSS138, SW1 CT2088-ND, U1 CYC1000, U2 MAX3232

Commit message: Starting layout
Parts:
- removed J5: Power connector, symbol Connector:Barrel_Jack_Switch
- added H1, H2, H3, H4: MountingHole, MountingHole:MountingHole_3.2mm_M3, symbol Mechanical:MountingHole
- added J5: Power, falco_terminal:BarrelJack_CUI_PJ-063AH_Horizontal, symbol Connector:Barrel_Jack_MountingPin
- C1, C2, C3, C4, C5, C6, C7, C8: footprint (none) -> Capacitor_SMD:C_0603_1608Metric_Pad1.08x0.95mm_HandSolder
- C9: footprint (none) -> Capacitor_SMD:C_1210_3225Metric_Pad1.33x2.70mm_HandSolder
- J1: value VGA Connector -> L77HDE15SD1CH4F-ND; footprint (none) -> falco_terminal:AMPHENOL_L77HDE15SD1CH4F; symbol Connector:DB15_Female_HighDensity_MountingHoles -> falco_terminal:DB15_Female
- J2: footprint (none) -> falco_terminal:CUI_MD-60SM
- J3: footprint (none) -> falco_terminal:AMPHENOL_LD09S33E4GX00LF; symbol Connector:DB9_Female_MountingHoles -> falco_terminal:DB9_Female
- J4: footprint (none) -> Connector_PinHeader_2.54mm:PinHeader_1x06_P2.54mm_Vertical
- R1, R10, R11, R12, R13, R14, R15, R16, R17, R18, R2, R3, R4, R5, R6, R7, R8, R9: footprint (none) -> Resistor_SMD:R_0603_1608Metric_Pad0.98x0.95mm_HandSolder
- SW1: footprint (none) -> Package_DIP:DIP-16_W7.62mm_Socket
- U1: footprint (none) -> falco_CYC1000:CYC1000
- U2: footprint (none) -> falco_terminal:TSSOP-16_4.4x5mm_P0.65mm
Connections:
- net GND: now also J1.S1, J1.S2, J3.S1, J3.S2, J5.2, J5.MP (MountPin); no longer J1.0, J3.0 (PAD)
- net VCC-5.0: now also J5.1
- no-connect marks 22 -> 21

Commit message: Wiring connectors
Parts:
- J2: symbol Connector:Mini-DIN-6 -> falco_terminal:Mini-DIN-6
Connections:
- net GND: now also J2.S1, J2.S2, J2.S3
Changed lines of the file:
@@
 $EndComp
 $Comp
-L Connector:Mini-DIN-6 J2
+L falco_terminal:Mini-DIN-6 J2
 U 1 1 604B68AC
 P 2700 4700
 F 0 "J2" H 2700 4950 50  0000 C CNN
-F 1 "Mini-DIN-6" H 2700 4450 50  0000 C CNN
+F 1 "Mini-DIN-6" H 2700 5050 50  0000 C CNN
 F 2 "falco_terminal:CUI_MD-60SM" H 2700 4700 50  0001 C CNN
 F 3 "http://service.powerdynamics.com/ec/Catalog17/Section%2011.pdf" H 2700 4700 50  0001 C CNN
@@
 $EndComp
 Wire Wire Line
-	2200 5250 2200 5350
+	2200 5250 2200 5300
 Text Notes 2100 3100 0    50   ~ 0
 PS-2 Keyboards run on 5 volts, and the signals are open-collector.\nWe so far have no reason to drive them, but we do have to\nlevel-shift them down to 3.3 volts for the FPGA.  Our level-shifters\nare bidirectional, so we can drive the keyboard, if we ever need to.\n\nThe keyboard provides the clock to the FPGA.
@@
 	1    0    0    -1
 $EndComp
+Wire Wire Line
+	2200 5300 2600 5300
+Wire Wire Line
+	2800 5300 2800 5000
+Connection ~ 2200 5300
+Wire Wire Line
+	2200 5300 2200 5350
+Wire Wire Line
+	2700 5000 2700 5300
+Connection ~ 2700 5300
+Wire Wire Line
+	2700 5300 2800 5300
+Wire Wire Line
+	2600 5000 2600 5300
+Connection ~ 2600 5300
+Wire Wire Line
+	2600 5300 2700 5300
 $EndSCHEMATC

Commit message: Should be pretty close
Parts:
- added C10: 0.1u, Capacitor_SMD:C_0603_1608Metric_Pad1.08x0.95mm_HandSolder, symbol Device:C
Connections:
- net +3V3: now also C10.1
- net GND: now also C10.2
- net PIXEL_B1: now also U1.2 (GP1_R12); no longer U1.6 (GP5_P14)
- net PIXEL_B2: now also U1.3 (GP2_T13); no longer U1.7 (GP6_R14)
- net PIXEL_R1: now also U1.6 (GP5_P14); no longer U1.2 (GP1_R12)
- net PIXEL_R2: now also U1.7 (GP6_R14); no longer U1.3 (GP2_T13)
Changed lines of the file:
@@
 NoConn ~ 6750 3400
 Text Label 6150 3500 0    50   ~ 0
-PIXEL_R1
+PIXEL_B1
 Text Label 6150 3600 0    50   ~ 0
-PIXEL_R2
+PIXEL_B2
 Text Label 6150 3700 0    50   ~ 0
 PIXEL_G1
@@
 PIXEL_G2
 Text Label 6150 3900 0    50   ~ 0
-PIXEL_B1
+PIXEL_R1
 Text Label 6150 4000 0    50   ~ 0
-PIXEL_B2
+PIXEL_R2
 Text Label 6150 4100 0    50   ~ 0
 HSYNC
@@
 Wire Wire Line
 	2600 5300 2700 5300
+$Comp
+L Device:C C10
+U 1 1 6050E6BE
+P 4050 4550
+F 0 "C10" H 4075 4650 50  0000 L CNN
+F 1 "0.1u" H 4075 4450 50  0000 L CNN
+F 2 "Capacitor_SMD:C_0603_1608Metric_Pad1.08x0.95mm_HandSolder" H 4088 4400 50  0001 C CNN
+F 3 "~" H 4050 4550 50  0001 C CNN
+	1    4050 4550
+	1    0    0    -1
+$EndComp
+$Comp
+L power:+3V3 #PWR0101
+U 1 1 605108D7
+P 4050 4350
+F 0 "#PWR0101" H 4050 4200 50  0001 C CNN
+F 1 "+3V3" H 4050 4490 50  0000 C CNN
+F 2 "" H 4050 4350 50  0001 C CNN
+F 3 "" H 4050 4350 50  0001 C CNN
+	1    4050 4350
+	1    0    0    -1
+$EndComp
+$Comp
+L power:GND #PWR0102
+U 1 1 60511003
+P 4050 4750
+F 0 "#PWR0102" H 4050 4500 50  0001 C CNN
+F 1 "GND" H 4050 4600 50  0000 C CNN
+F 2 "" H 4050 4750 50  0001 C CNN
+F 3 "" H 4050 4750 50  0001 C CNN
+	1    4050 4750
+	1    0    0    -1
+$EndComp
+Wire Wire Line
+	4050 4350 4050 4400
+Wire Wire Line
+	4050 4700 4050 4750
 $EndSCHEMATC

Commit message: V1 looks good
Parts:
- added R19, R20: 100, Resistor_SMD:R_0603_1608Metric_Pad0.98x0.95mm_HandSolder, symbol Device:R_US
- H1, H2, H3, H4: value MountingHole -> MountingHole_Pad; footprint MountingHole:MountingHole_3.2mm_M3 -> MountingHole:MountingHole_3.2mm_M3_DIN965_Pad; symbol Mechanical:MountingHole -> Mechanical:MountingHole_Pad
Connections:
- net GND: now also H1.1, H2.1, H3.1, H4.1
- net HSYNC: now also R19.1; no longer J1.13
- net VSYNC: now also R20.1; no longer J1.14
- net C1+: now reaches C4.1, U2.1 (C1+)
- net VS+: now reaches C7.1, U2.2 (VS+)
- net C1-: now reaches C4.2, U2.3 (C1-)
- net C2+: now reaches C5.1, U2.4 (C2+)
- net C2-: now reaches C5.2, U2.5 (C2-)
- net VS-: now reaches C6.1, U2.6 (VS-)
- new net: J1.13, R19.2
- new net: J1.14, R20.2
Changed lines of the file:
@@
 U 1 1 604D2444
 P 11700 5500
-F 0 "C4" H 11725 5600 50  0000 L CNN
-F 1 "0.1u" H 11725 5400 50  0000 L CNN
+F 0 "C4" H 11550 5600 50  0000 L CNN
+F 1 "0.1u" H 11500 5400 50  0000 L CNN
 F 2 "Capacitor_SMD:C_0603_1608Metric_Pad1.08x0.95mm_HandSolder" H 11738 5350 50  0001 C CNN
 F 3 "~" H 11700 5500 50  0001 C CNN
@@
 NoConn ~ 14250 3000
 Wire Wire Line
-	15050 2600 14250 2600
-Wire Wire Line
-	15050 2800 14250 2800
-Text Label 15050 2600 2    50   ~ 0
+	15450 2600 14650 2600
+Wire Wire Line
+	15450 2800 14650 2800
+Text Label 15450 2600 2    50   ~ 0
 HSYNC
-Text Label 15050 2800 2    50   ~ 0
+Text Label 15450 2800 2    50   ~ 0
 VSYNC
 $Comp
@@
 Connection ~ 2650 8500
 $Comp
-L Mechanical:MountingHole H1
+L Mechanical:MountingHole_Pad H1
 U 1 1 605CE31F
 P 2700 9850
 F 0 "H1" H 2700 10050 50  0000 C CNN
-F 1 "MountingHole" H 2700 9975 50  0001 C CNN
-F 2 "MountingHole:MountingHole_3.2mm_M3" H 2700 9850 50  0001 C CNN
+F 1 "MountingHole_Pad" H 2700 9975 50  0001 C CNN
+F 2 "MountingHole:MountingHole_3.2mm_M3_DIN965_Pad" H 2700 9850 50  0001 C CNN
 F 3 "~" H 2700 9850 50  0001 C CNN
 	1    2700 9850
@@
 $EndComp
 $Comp
-L Mechanical:MountingHole H2
+L Mechanical:MountingHole_Pad H2
 U 1 1 605D1927
 P 3050 9850
 F 0 "H2" H 3050 10050 50  0000 C CNN
-F 1 "MountingHole" H 3050 9975 50  0001 C CNN
-F 2 "MountingHole:MountingHole_3.2mm_M3" H 3050 9850 50  0001 C CNN
+F 1 "MountingHole_Pad" H 3050 9975 50  0001 C CNN
+F 2 "MountingHole:MountingHole_3.2mm_M3_DIN965_Pad" H 3050 9850 50  0001 C CNN
 F 3 "~" H 3050 9850 50  0001 C CNN
 	1    3050 9850
@@
 $EndComp
 $Comp
-L Mechanical:MountingHole H3
+L Mechanical:MountingHole_Pad H3
 U 1 1 605D1BDF
 P 3400 9850
 F 0 "H3" H 3400 10050 50  0000 C CNN
-F 1 "MountingHole" H 3400 9975 50  0001 C CNN
-F 2 "MountingHole:MountingHole_3.2mm_M3" H 3400 9850 50  0001 C CNN
+F 1 "MountingHole_Pad" H 3400 9975 50  0001 C CNN
+F 2 "MountingHole:MountingHole_3.2mm_M3_DIN965_Pad" H 3400 9850 50  0001 C CNN
 F 3 "~" H 3400 9850 50  0001 C CNN
 	1    3400 9850
@@
 $EndComp
 $Comp
-L Mechanical:MountingHole H4
+L Mechanical:MountingHole_Pad H4
 U 1 1 605D1D93
 P 3750 9850
 F 0 "H4" H 3750 10050 50  0000 C CNN
-F 1 "MountingHole" H 3750 9975 50  0001 C CNN
-F 2 "MountingHole:MountingHole_3.2mm_M3" H 3750 9850 50  0001 C CNN
+F 1 "MountingHole_Pad" H 3750 9975 50  0001 C CNN
+F 2 "MountingHole:MountingHole_3.2mm_M3_DIN965_Pad" H 3750 9850 50  0001 C CNN
 F 3 "~" H 3750 9850 50  0001 C CNN
 	1    3750 9850
@@
 Wire Wire Line
 	4050 4700 4050 4750
+$Comp
+L Device:R_US R19
+U 1 1 60518B55
+P 14500 2600
+F 0 "R19" V 14400 2700 50  0000 C CNN
+F 1 "100" V 14400 2500 50  0000 C CNN
+F 2 "Resistor_SMD:R_0603_1608Metric_Pad0.98x0.95mm_HandSolder" V 14540 2590 50  0001 C CNN
+F 3 "~" H 14500 2600 50  0001 C CNN
+	1    14500 2600
+	0    1    1    0
+$EndComp
+$Comp
+L Device:R_US R20
+U 1 1 605195CB
+P 14500 2800
+F 0 "R20" V 14400 2900 50  0000 C CNN
+F 1 "100" V 14400 2700 50  0000 C CNN
+F 2 "Resistor_SMD:R_0603_1608Metric_Pad0.98x0.95mm_HandSolder" V 14540 2790 50  0001 C CNN
+F 3 "~" H 14500 2800 50  0001 C CNN
+	1    14500 2800
+	0    1    1    0
+$EndComp
+Wire Wire Line
+	14250 2600 14350 2600
+Wire Wire Line
+	14250 2800 14350 2800
+Text Label 13550 5850 0    50   ~ 0
+VS+
+Text Label 13550 6150 0    50   ~ 0
+VS-
+Text Label 13500 5350 0    50   ~ 0
+C2+
+Text Label 13500 5650 0    50   ~ 0
+C2-
+Text Label 11700 5350 0    50   ~ 0
+C1+
+Text Label 11700 5650 0    50   ~ 0
+C1-
+$Comp
+L power:GND #PWR0103
+U 1 1 6054131C
+P 2700 10100
+F 0 "#PWR0103" H 2700 9850 50  0001 C CNN
+F 1 "GND" H 2700 9950 50  0000 C CNN
+F 2 "" H 2700 10100 50  0001 C CNN
+F 3 "" H 2700 10100 50  0001 C CNN
+	1    2700 10100
+	1    0    0    -1
+$EndComp
+Wire Wire Line
+	2700 10100 2700 10050
+Wire Wire Line
+	2700 10050 3050 10050
+Wire Wire Line
+	3750 10050 3750 9950
+Connection ~ 2700 10050
+Wire Wire Line
+	2700 10050 2700 9950
+Wire Wire Line
+	3400 9950 3400 10050
+Connection ~ 3400 10050
+Wire Wire Line
+	3400 10050 3750 10050
+Wire Wire Line
+	3050 9950 3050 10050
+Connection ~ 3050 10050
+Wire Wire Line
+	3050 10050 3400 10050
 $EndSCHEMATC

Commit message: Sense of RX/TX and CTS/RTS were backwards.
Fortunately, that is easy to fix in the FPGA by remapping the signals to
different pins.
Connections:
- net UART_CTS: now also U1.29 (GP22_R1), U2.9 (R2OUT); no longer U1.30 (GP21_P1), U2.10 (T2IN)
- net UART_RTS: now also U1.30 (GP21_P1), U2.10 (T2IN); no longer U1.29 (GP22_R1), U2.9 (R2OUT)
- net UART_RX: now also U1.11 (GP10_L16), U2.12 (R1OUT); no longer U1.10 (GP9_L15), U2.11 (T1IN)
- net UART_TX: now also U1.10 (GP9_L15), U2.11 (T1IN); no longer U1.11 (GP10_L16), U2.12 (R1OUT)
Other:
- note added: "Signal names at the J3 UART Connector are named from the perspective\nof the DTE to which we are connected, and are therefore backwards\nwith respect to our FPGA!\n\nWe are wired as a DCE (i.e., like a modem). We connect to a DTE (PC or\nother computer) with a straight cable. However, the PiDP-11 is also\nwired as a DCE, so we need a null-modem cable with it.\n\nWe receive data from the DTE on pi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"
Changed lines of the file:
@@
 	11250 6950 11900 6950
 Text Label 11250 6350 0    50   ~ 0
+UART_TX
+Text Label 11250 6550 0    50   ~ 0
+UART_RTS
+Text Label 11250 6750 0    50   ~ 0
 UART_RX
-Text Label 11250 6550 0    50   ~ 0
+Text Label 11250 6950 0    50   ~ 0
 UART_CTS
-Text Label 11250 6750 0    50   ~ 0
-UART_TX
-Text Label 11250 6950 0    50   ~ 0
-UART_RTS
 $Comp
 L falco_terminal:DB15_Female J1
@@
 VSYNC
 Text Label 6150 4400 0    50   ~ 0
+UART_TX
+Text Label 6150 4500 0    50   ~ 0
 UART_RX
-Text Label 6150 4500 0    50   ~ 0
-UART_TX
 Text Label 6150 4600 0    50   ~ 0
 KBD_CLK
@@
 DIP_SW3
 Text Label 8500 4700 2    50   ~ 0
+UART_CTS
+Text Label 8500 4800 2    50   ~ 0
 UART_RTS
-Text Label 8500 4800 2    50   ~ 0
-UART_CTS
 $Comp
 L Switch:SW_DIP_x08 SW1
@@
 Wire Wire Line
 	3050 10050 3400 10050
+Text Notes 11900 9150 0    50   ~ 0
+Signal names at the J3 UART Connector are named from the perspective\nof the DTE to which we are connected, and are therefore backwards\nwith respect to our FPGA!\n\nWe are wired as a DCE (i.e., like a modem).  We connect to a DTE (PC or\nother computer) with a straight cable.  However, the PiDP-11 is also\nwired as a DCE, so we need a null-modem cable with it.\n\nWe receive data from the DTE on pin 3 (DTE TXD becomes our\nUART_RX), and we transmit data to the DTE on pin 2 (our UART_TX\nbecomes DTE RXD).\n\nSimilarly, our UART_RTS signal becomes the DTE CTS signal on pin 8,\nand the DTS RTS signal on pin 7 becomes our UART_CTS signal.\n\nWe deassert our UART_RTS when our receive buffer becomes too full.
 $EndSCHEMATC

Commit message: Fix R values & silk
Parts:
- R1, R3, R5: value 500 -> 499
Changed lines of the file:
@@
 P 10150 2200
 F 0 "R1" V 10050 2300 50  0000 C CNN
-F 1 "500" V 10050 2100 50  0000 C CNN
+F 1 "499" V 10050 2100 50  0000 C CNN
 F 2 "Resistor_SMD:R_0603_1608Metric_Pad0.98x0.95mm_HandSolder" V 10190 2190 50  0001 C CNN
 F 3 "~" H 10150 2200 50  0001 C CNN
@@
 P 10150 2700
 F 0 "R3" V 10050 2800 50  0000 C CNN
-F 1 "500" V 10050 2600 50  0000 C CNN
+F 1 "499" V 10050 2600 50  0000 C CNN
 F 2 "Resistor_SMD:R_0603_1608Metric_Pad0.98x0.95mm_HandSolder" V 10190 2690 50  0001 C CNN
 F 3 "~" H 10150 2700 50  0001 C CNN
@@
 P 10150 3200
 F 0 "R5" V 10050 3300 50  0000 C CNN
-F 1 "500" V 10050 3100 50  0000 C CNN
+F 1 "499" V 10050 3100 50  0000 C CNN
 F 2 "Resistor_SMD:R_0603_1608Metric_Pad0.98x0.95mm_HandSolder" V 10190 3190 50  0001 C CNN
 F 3 "~" H 10150 3200 50  0001 C CNN
